File: PCB/SDR.kicad_pcb (KiCad board)
At the start: 4 copper layers, 158.8 x 71.3 mm, 219 parts, among them IC1 RFSW6042TR7, IC2 RFSW6042TR7, IC5 CMX992Q3, J1 SMA, J11 SMA, J12 SMA, J13 Nucleo_GPIO, J14 SMA, J15 Nucleo_GPIO, J2 Nucleo_GPIO, J3 Nucleo_GPIO, J4 Nucleo_GPIO, J5 FPGA, J6 Tang Nano, J7 Tang Nano, J8 Tang Nano, J9 USB_C_Receptacle_PowerOnly_6P, U1 SGL0622Z, U10 ECS-45K15B, U2 ADF4351BCPZ-RL7, U3 ATX-H12-F-10.000MHZ-F25-T, U4 MASWSS0115, U6 LTC2323CUFD-12-PBF, U7 LT1762-2.5, U8 LT1962-3.3, U9 ECS-45K15B

Commit message: Add files via upload
Parts:
- removed TP1: SCK-, TestPoint:TestPoint_Pad_D3.0mm
- removed TP2: SCK+, TestPoint:TestPoint_Pad_D3.0mm
- added J10: Tang Nano, Connector_Wire:SolderWire-0.25sqmm_1x03_P4.5mm_D0.65mm_OD2mm, F.Cu at (235.5, 135.1)
Routing:
- net /SCK-: track 17.6 -> 25.4 mm
- net /SCK+: track 18.3 -> 25.4 mm

Commit message: Add files via upload
Routing:
- net GND: track 172.9 -> 176.0 mm, vias 265 -> 267
